File: PCB/_autosave-canctrl.kicad_sch (KiCad schematic)
At the start: 18 parts, among them U4 SN65HVD230DR, U5 MCP2515-xSO, Y2 ABM8-16.000MHZ-B2-T

Commit message: Redo time, pcb too close
Parts:
- Y2: footprint ABM8-16.000MHZ-B2-T-Alt:XTAL_ABM8-16.000MHZ-B2-T -> ABM8-16.000MHZ-B2-T:XTAL_ABM8-16.000MHZ-B2-T
Changed lines of the file:
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@@
 			)
 		)
-		(property "Footprint" "ABM8-16.000MHZ-B2-T-Alt:XTAL_ABM8-16.000MHZ-B2-T"
+		(property "Footprint" "ABM8-16.000MHZ-B2-T:XTAL_ABM8-16.000MHZ-B2-T"
 			(at 50.8 86.36 0)
 			(effects
