File: PCB/PixAppleV1.1.kicad_pcb (KiCad board)
At the start: 4 copper layers, 50 x 35 mm, 78 parts, among them J1 USB_C_Receptacle_USB2.0_16P, J2 Conn_01x02_Pin, J3 Conn_01x02_Pin, J5 Conn_02x08_Odd_Even, J7 Conn_01x02_Pin, U1 RP2040, U2 W25Q128JVS, U3 NCP1117-3.3_SOT223, U4 MCP2515-xSO, U6 TCAN337G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

Commit message: BOM will finish soon
Other:
- board text added: "16"
- board text added: "18"
- board text added: "20"
- board text added: "22"
- board text added: "24"
- board text added: "26"
- board text added: "28"
- board text added: "29"
- board text added: "3V3"
- board text added: "G"
Changed lines of the file:
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@@
 		(tags "Through hole pin header THT 2x08 2.54mm double row")
 		(property "Reference" "J5"
-			(at 3.59 -2.46 0)
+			(at 4.09 20.24 0)
 			(layer "F.SilkS")
 			(effects
@@
 				(font
 					(size 1 1)
-					(thickness 0.15)
+					(thickness 0.2)
+					(bold yes)
 				)
 			)
@@
 				(font
 					(size 1 1)
-					(thickness 0.15)
+					(thickness 0.2)
+					(bold yes)
 				)
 			)
@@
 		(layer "Edge.Cuts")
 	)
+	(gr_text "29"
+		(at 166.3 85.9 0)
+		(layer "F.SilkS")
+		(effects
+			(font
+				(size 1 1)
+				(thickness 0.2)
+				(bold yes)
+			)
+			(justify left bottom)
+		)
+	)
+	(gr_text "28"
+		(at 162.8 91.3 90)
+		(layer "F.SilkS")
+		(effects
+			(font
+				(size 1 1)
+				(thickness 0.2)
+				(bold yes)
+			)
+			(justify left bottom)
+		)
+	)
+	(gr_text "3V3"
+		(at 163.1 86 0)
+		(layer "F.SilkS")
+		(effects
+			(font
+				(size 1 1)
+				(thickness 0.2)
+				(bold yes)
+			)
+			(justify left bottom)
+		)
+	)
 	(gr_text "RST"
 		(at 139.9 76.6 0)
@@
 		)
 	)
+	(gr_text "G"
+		(at 166.8 108.7 0)
+		(layer "F.SilkS")
+		(effects
+			(font
+				(size 1 1)
+				(thickness 0.2)
+				(bold yes)
+			)
+			(justify left bottom)
+		)
+	)
+	(gr_text "24"
+		(at 162.8 96.5 90)
+		(layer "F.SilkS")
+		(effects
+			(font
+				(size 1 1)
+				(thickness 0.2)
+				(bold yes)
+			)
+			(justify left bottom)
+		)
+	)
+	(gr_text "16"
+		(at 163.5 108.8 0)
+		(layer "F.SilkS")
+		(effects
+			(font
+				(size 1 1)
+				(thickness 0.2)
+				(bold yes)
+			)
+			(justify left bottom)
+		)
+	)
+	(gr_text "20"
+		(at 162.8 101.7 90)
+		(layer "F.SilkS")
+		(effects
+			(font
+				(size 1 1)
+				(thickness 0.2)
+				(bold yes)
+			)
+			(justify left bottom)
+		)
+	)
+	(gr_text "26"
+		(at 162.8 94 90)
+		(layer "F.SilkS")
+		(effects
+			(font
+				(size 1 1)
+				(thickness 0.2)
+				(bold yes)
+			)
+			(justify left bottom)
+		)
+	)
 	(gr_text "(G)"
 		(at 120.75 86.85 0)
@@
 		)
 	)
+	(gr_text "22"
+		(at 162.8 99 90)
+		(layer "F.SilkS")
+		(effects
+			(font
+				(size 1 1)
+				(thickness 0.2)
+				(bold yes)
+			)
+			(justify left bottom)
+		)
+	)
+	(gr_text "18"
+		(at 162.8 104.2 90)
+		(layer "F.SilkS")
+		(effects
+			(font
+				(size 1 1)
+				(thickness 0.2)
+				(bold yes)
+			)
+			(justify left bottom)
+		)
+	)
 	(gr_text "PixAppleV1.1"
 		(at 137.65 106.3 -0)
@@
 	)
 	(via
-		(at 121.75 106.25)
+		(at 123 105.1)
 		(size 0.6)
 		(drill 0.3)
@@
 	)
 	(via
-		(at 122.3 108.1)
+		(at 123.1 108.5)
 		(size 0.6)
 		(drill 0.3)
@@
 	)
 	(via
-		(at 121.75 104.5)
+		(at 123.1 106.9)
 		(size 0.6)
 		(drill 0.3)
@@
 	)
 	(segment
+		(start 159.711074 107.5)
+		(end 156.25 107.5)
+		(width 0.5)
+		(layer "B.Cu")
+		(net 2)
+	)
+	(segment
 		(start 151.371389 92.275)
 		(end 152.134889 91.5115)
@@
 	)
 	(segment
+		(start 162.501 103.902)
+		(end 162.501 104.710074)
+		(width 0.5)
+		(layer "B.Cu")
+		(net 2)
+	)
+	(segment
 		(start 155.251 106.501)
 		(end 148.051 106.501)
@@
 	)
 	(segment
+		(start 159.35 100.751)
+		(end 162.501 103.902)
+		(width 0.5)
+		(layer "B.Cu")
+		(net 2)
+	)
+	(segment
 		(start 145.5 83.5)
 		(end 143 83.5)
@@
 	)
 	(segment
-		(start 159.711075 107.5)
-		(end 156.25 107.5)
-		(width 0.5)
-		(layer "B.Cu")
-		(net 2)
-	)
-	(segment
 		(start 154.2625 106.501)
 		(end 155.251 106.501)
@@
 	)
 	(segment
-		(start 162.501 104.710075)
-		(end 159.711075 107.5)
-		(width 0.5)
-		(layer "B.Cu")
-		(net 2)
-	)
-	(segment
 		(start 135.412925 84.75)
 		(end 141.75 84.75)
@@
 	)
 	(segment
-		(start 159.35 100.751)
-		(end 162.501 103.902)
-		(width 0.5)
-		(layer "B.Cu")
-		(net 2)
-	)
-	(segment
 		(start 144.716763 100.751)
 		(end 144.757802 100.709961)
@@
 	)
 	(segment
+		(start 162.501 104.710074)
+		(end 159.711074 107.5)
+		(width 0.5)
+		(layer "B.Cu")
+		(net 2)
+	)
+	(segment
 		(start 145.5 83.5)
 		(end 149.056082 87.056082)
@@
 		(width 0.5)
 		(layer "B.Cu")
-		(net 2)
-	)
-	(segment
-		(start 162.501 103.902)
-		(end 162.501 104.710075)
-		(width 0.5)
-		(layer "B.Cu")
